File: rig/electrical/TeensyOpenLoop/TeensyOpenLoop.kicad_pcb (KiCad board)
At the start: 2 copper layers, 111.1 x 86 mm, 25 parts, among them J1 TST-104-01-G-D, J2 TST-103-03-T-D, J3 TST-102-01-G-D, J5 PJ-002B, J6 TST-105-01-X-D, J7 PJ-002B, U1 Teensy4.1, U2 SN74LVC245AN, U3 SN74AHCT125N, U4 SN74AHCT125N, U6 SN74LVC245AN

Commit message: updates to electrical
Other:
- board text added: "SN54AHCT125"
- board text removed: "SN74LVC245A"
Changed lines of the file:
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@@
 		)
 	)
-	(gr_text "SN74LVC245A"
+	(gr_text "SN54AHCT125"
 		(at 196.342 103.378 0)
 		(layer "F.SilkS")
@@
 		)
 	)
-	(gr_text "SN74LVC245A"
+	(gr_text "SN54AHCT125"
 		(at 148.336 105.918 0)
 		(layer "F.SilkS")
